File: MMDVM_Pi3_Hat.sch (KiCad schematic (older format))
At the start: 91 parts, among them J1 USB_B_Mini, J2 I2C, J3 STLink, J4 Display, J5 SMA, J6 Conn_02x09_Counter_Clockwise, P1 Pi3, U1 LM1117MPX-3.3, U2 STM32F103C8T6, U3 ADF7021, U4 OSHW-Logo_19x20mm, U5 MMDVM-Logo, U6 KiCAD-Logo_6mm, U7 CC_BY_NC_SA, X1 ECS-TXO-5032-147.4-TR, Y1 8MHz

Commit message: Start PCB Layout
Parts:
- removed J6: Conn_02x09_Counter_Clockwise, Connector_PinSocket_2.54mm:PinSocket_2x09_P2.54mm_Vertical, symbol Connector_Generic:Conn_02x09_Counter_Clockwise
- added J6: Conn_02x10_Counter_Clockwise, Connector_PinHeader_2.54mm:PinHeader_2x10_P2.54mm_Vertical, symbol Connector_Generic:Conn_02x10_Counter_Clockwise
Connections:
- net labels added: +3V3
- net labels removed: RF, VDD
- wire segments 392 -> 395
Other:
- note removed: "Antenna"
