File: MMDVM_Pi3_Hat.kicad_pcb (KiCad board)
At the start: 2 copper layers, 65 x 56 mm, 91 parts, among them J1 USB_B_Mini, J2 I2C, J3 STLink, J4 Display, J5 SMA, J6 Conn_02x09_Counter_Clockwise, P1 Pi3, U1 LM1117MPX-3.3, U2 STM32F103C8T6, U3 ADF7021, U4 OSHW-Logo_19x20mm, U5 MMDVM-Logo, U6 KiCAD-Logo_6mm, U7 CC_BY_NC_SA, X1 ECS-TXO-5032-147.4-TR, Y1 8MHz

Commit message: Start PCB Layout
Parts:
- J6: value Conn_02x09_Counter_Clockwise -> Conn_02x10_Counter_Clockwise; footprint Connector_PinSocket_2.54mm:PinSocket_2x09_P2.54mm_Vertical -> Connector_PinHeader_2.54mm:PinHeader_2x10_P2.54mm_Vertical
- U4: moved to B.Cu
- moved U7 157.4 mm to (209.5, 162.5)
- moved L5 151.9 mm to (214.2, 138.3)
- moved L4 151.7 mm to (209.1, 135.8)
- moved C29 149.5 mm to (214.2, 135.8)
- moved C30 137.7 mm to (223.9, 135.8), turned to 180 degrees
- moved L6 133.7 mm to (223.9, 138.3), turned to 180 degrees
- moved C26 125.5 mm to (219.3, 138.3), turned to 180 degrees
- moved J1 78.2 mm to (247.2, 146.4)
- moved L1 72.4 mm to (279.5, 163.0)
- moved U6 72.2 mm to (239.6, 109.4)
- moved J6 62.6 mm to (258.4, 108.3)
- moved C4 56.4 mm to (287.6, 169.0)
- moved C3 56.0 mm to (269.4, 173.5)
- moved C6 55.8 mm to (278.4, 169.5)
- moved C5 51.1 mm to (278.5, 175.0)
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Connections:
- net RF renamed Net-(C7-Pad1)
- C10 pad 2: VDD -> +3V3
- C11 pad 1: VDD -> +3V3
- C14 pad 2: VDD -> +3V3
- C16 pad 1: VDD -> +3V3
- C20 pad 1: VDD -> +3V3
- C21 pad 1: VDD -> +3V3
- C22 pad 1: VDD -> +3V3
- C28 pad 1: VDD -> +3V3
- C31 pad 1: VDD -> +3V3
- C5 pad 1: VDD -> +3V3
- C6 pad 1: VDD -> +3V3
- C9 pad 2: VDD -> +3V3
- J2 pad 1: VDD -> +3V3
- J3 pad 1: VDD -> +3V3
- J6 pad 10: CLK_OUT -> GND
- J6 pad 11: SW_CLK -> GND
- J6 pad 12: SW_DIO -> CLK_OUT
- J6 pad 13: USB_DP -> SW_CLK
- J6 pad 14: USB_DM -> SW_DIO
- J6 pad 15: TXD -> USB_DP
- J6 pad 16: RXD -> USB_DM
- J6 pad 17: SCL -> TXD
- J6 pad 18: SDA -> RXD
- J6 pad 2: VDD -> +3V3
- L1 pad 2: VDD -> +3V3
- L3 pad 2: VDD -> +3V3
- P1 pad 11: (no net) -> /GPIO17(GEN0)
- P1 pad 12: (no net) -> /GPIO18(GEN1)(PWM0)
- P1 pad 13: (no net) -> /GPIO27(GEN2)
- P1 pad 15: (no net) -> /GPIO22(GEN3)
- P1 pad 16: (no net) -> /GPIO23(GEN4)
- P1 pad 18: (no net) -> /GPIO24(GEN5)
- P1 pad 19: (no net) -> /GPIO10(SPI0_MOSI)
- P1 pad 21: (no net) -> /GPIO9(SPI0_MISO)
- P1 pad 22: (no net) -> /GPIO25(GEN6)
- P1 pad 23: (no net) -> /GPIO11(SPI0_SCK)
- P1 pad 24: (no net) -> /GPIO8(SPI0_CE_N)
- P1 pad 26: (no net) -> /GPIO7(SPI1_CE_N)
- P1 pad 27: (no net) -> /ID_SD
- P1 pad 28: (no net) -> /ID_SC
- P1 pad 29: (no net) -> /GPIO5
- P1 pad 31: (no net) -> /GPIO6
- P1 pad 32: (no net) -> /GPIO12(PWM0)
- P1 pad 33: (no net) -> /GPIO13(PWM1)
- P1 pad 35: (no net) -> /GPIO19(SPI1_MISO)
- P1 pad 36: (no net) -> /GPIO16
- P1 pad 37: (no net) -> /GPIO26
- P1 pad 7: (no net) -> /GPIO4(GCLK)
- R2 pad 2: VDD -> +3V3
- R3 pad 2: VDD -> +3V3
- R5 pad 2: VDD -> +3V3
- U2 pad 1: VDD -> +3V3
- U2 pad 10: (no net) -> Net-(U2-Pad10)
- U2 pad 11: (no net) -> Net-(U2-Pad11)
- U2 pad 14: (no net) -> Net-(U2-Pad14)
- U2 pad 15: (no net) -> Net-(U2-Pad15)
- U2 pad 16: (no net) -> Net-(U2-Pad16)
- U2 pad 17: (no net) -> Net-(U2-Pad17)
- U2 pad 21: (no net) -> Net-(U2-Pad21)
- U2 pad 22: (no net) -> Net-(U2-Pad22)
- U2 pad 24: VDD -> +3V3
- U2 pad 36: VDD -> +3V3
- U2 pad 4: (no net) -> Net-(U2-Pad4)
- U2 pad 46: (no net) -> Net-(U2-Pad46)
- U2 pad 48: VDD -> +3V3
- U2 pad 9: VDD -> +3V3
- U3 pad 13: (no net) -> Net-(U3-Pad13)
- U3 pad 14: (no net) -> Net-(U3-Pad14)
- U3 pad 15: (no net) -> Net-(U3-Pad15)
- U3 pad 16: (no net) -> Net-(U3-Pad16)
- U3 pad 17: (no net) -> Net-(U3-Pad17)
- U3 pad 18: (no net) -> Net-(U3-Pad18)
- U3 pad 20: (no net) -> Net-(U3-Pad20)
- U3 pad 21: (no net) -> Net-(U3-Pad21)
- U3 pad 23: (no net) -> Net-(U3-Pad23)
- U3 pad 3: VDD -> +3V3
- U3 pad 30: (no net) -> Net-(U3-Pad30)
- U3 pad 32: VDD -> +3V3
- U3 pad 33: (no net) -> Net-(U3-Pad33)
- U3 pad 37: (no net) -> Net-(U3-Pad37)
- U3 pad 38: (no net) -> Net-(U3-Pad38)
- U3 pad 40: VDD -> +3V3
- U3 pad 43: VDD -> +3V3
- U3 pad 9: VDD -> +3V3
- X1 pad 1: (no net) -> Net-(X1-Pad1)
- X1 pad 4: VDD -> +3V3
Routing:
- net +5V: track 0.00 -> 127.2 mm, vias 0 -> 2
- net Net-(C25-Pad2): track 0.00 -> 6.56 mm
- net Net-(C29-Pad1): track 0.00 -> 5.92 mm
- net Net-(C7-Pad1): track 0.00 -> 3.56 mm
- net Net-(C26-Pad1): track 0.00 -> 2.87 mm
- net Net-(C30-Pad1): track 0.00 -> 2.54 mm
- net Net-(C7-Pad2): track 6.22 -> 7.11 mm
Other:
- outline, holes or cut-outs redrawn

Commit message: Save
Parts:
- moved R22 176.2 mm to (198.2, 186.3)
- moved R21 174.8 mm to (198.2, 181.8)
- moved L2 171.2 mm to (206.3, 175.3), turned to 90 degrees
- moved R20 163.1 mm to (217.8, 184.0), turned to 180 degrees
- moved C31 157.8 mm to (198.2, 184.0), turned to 180 degrees
- moved C19 155.9 mm to (211.4, 175.3), turned to 270 degrees
- moved C16 149.2 mm to (222.4, 179.2), turned to 270 degrees
- moved C27 147.5 mm to (217.7, 186.1), turned to 180 degrees
- moved R18 141.7 mm to (217.8, 180.0), turned to 180 degrees
- moved C15 139.8 mm to (214.5, 175.7), turned to 180 degrees
- moved C32 132.2 mm to (206.1, 188.6)
- moved R19 124.9 mm to (217.8, 182.0), turned to 180 degrees
- moved C11 119.5 mm to (208.9, 175.3), turned to 90 degrees
- moved C28 119.5 mm to (224.4, 179.2), turned to 270 degrees
- moved X1 90.5 mm to (220.7, 173.1), turned to 180 degrees
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Routing:
- net +3V3: track 0.00 -> 35.4 mm, vias 0 -> 3
- net S_DATA: track 0.00 -> 16.5 mm, vias 0 -> 2
- net S_READ: track 0.00 -> 16.5 mm, vias 0 -> 2
- net S_CLK: track 0.00 -> 16.3 mm, vias 0 -> 2
- net SLE: track 0.00 -> 16.1 mm, vias 0 -> 2
- net GND: track 0.00 -> 12.8 mm, vias 0 -> 2
- net CLK_OUT: track 0.00 -> 11.2 mm
- net DATA_OUT: track 0.00 -> 10.7 mm
- net DATA_IN: track 0.00 -> 10.5 mm
- net Net-(R21-Pad2): track 0.00 -> 7.58 mm
- net Net-(R22-Pad2): track 0.00 -> 7.57 mm
- net Net-(C27-Pad2): track 0.00 -> 6.78 mm
- net Net-(C30-Pad1): track 2.54 -> 9.22 mm
- net Net-(L2-Pad2): track 0.00 -> 6.31 mm
- net Net-(R20-Pad2): track 0.00 -> 5.90 mm
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Other:
- rule via_min_drill: 0.3 -> 0.2
